Commit message: Update gripper control

File: urdf/aidal_eg2-4c2.urdf (robot description, URDF)
Before this commit: robot RealMan_AIDAL, 55 links, 54 joints
Links:
- link left_4C2_Link1: mass 0.0024292 -> 0.03; geometry visual mesh filename=package://aidal_description/meshes/EG2-4C2/4C2_Link1.STL
- link left_4C2_Link2: mass 0.0038971 -> 0.03; geometry collision box size=0.02 0.03 0.03; visual mesh filename=package://aidal_description/meshes/EG2-4C2/4C2_Link2.STL
- link left_4C2_Link3: mass 0.0038971 -> 0.03; geometry collision box size=0.02 0.03 0.03; visual mesh filename=package://aidal_description/meshes/EG2-4C2/4C2_Link3.STL
- link left_4C2_Link4: mass 0.0024292 -> 0.03; geometry visual mesh filename=package://aidal_description/meshes/EG2-4C2/4C2_Link4.STL
- link left_4C2_Link5: mass 0.0045068 -> 0.03; geometry collision box size=0.02 0.03 0.02; visual mesh filename=package://aidal_description/meshes/EG2-4C2/4C2_Link5.STL
- link left_4C2_Link6: mass 0.0045068 -> 0.03; geometry collision box size=0.02 0.03 0.02; visual mesh filename=package://aidal_description/meshes/EG2-4C2/4C2_Link6.STL
- link left_4C2_baselink: mass 0.072633 -> 0.05; geometry collision box size=0.08 0.03 0.12; visual mesh filename=package://aidal_description/meshes/EG2-4C2/4C2_baselink.STL
- link right_4C2_Link1: mass 0.0024292 -> 0.03; geometry visual mesh filename=package://aidal_description/meshes/EG2-4C2/4C2_Link1.STL
- link right_4C2_Link2: mass 0.0038971 -> 0.03; geometry collision box size=0.02 0.03 0.03; visual mesh filename=package://aidal_description/meshes/EG2-4C2/4C2_Link2.STL
- link right_4C2_Link3: mass 0.0038971 -> 0.03; geometry collision box size=0.02 0.03 0.03; visual mesh filename=package://aidal_description/meshes/EG2-4C2/4C2_Link3.STL
- link right_4C2_Link4: mass 0.0024292 -> 0.03; geometry visual mesh filename=package://aidal_description/meshes/EG2-4C2/4C2_Link4.STL
- link right_4C2_Link5: mass 0.0045068 -> 0.03; geometry collision box size=0.02 0.03 0.02; visual mesh filename=package://aidal_description/meshes/EG2-4C2/4C2_Link5.STL
- link right_4C2_Link6: mass 0.0045068 -> 0.03; geometry collision box size=0.02 0.03 0.02; visual mesh filename=package://aidal_description/meshes/EG2-4C2/4C2_Link6.STL
- link right_4C2_baselink: mass 0.072633 -> 0.05; geometry collision box size=0.08 0.03 0.12; visual mesh filename=package://aidal_description/meshes/EG2-4C2/4C2_baselink.STL
Joints:
- joint left_4C2_Joint2: limit lower=0 upper=0.82 effort=1 velocity=1 -> lower=0 upper=0.82 effort=50 velocity=1
- joint left_4C2_Joint3: limit lower=-0.82 upper=0 effort=1 velocity=1 -> lower=-0.82 upper=0 effort=50 velocity=1
- joint left_4C2_Joint4: limit lower=-0.82 upper=0 effort=1 velocity=1 -> lower=-0.82 upper=0 effort=50 velocity=1
- joint left_4C2_Joint5: limit lower=0 upper=0.82 effort=1 velocity=1 -> lower=0 upper=0.82 effort=50 velocity=1
- joint left_4C2_Joint6: limit lower=0 upper=0.82 effort=1 velocity=1 -> lower=0 upper=0.82 effort=50 velocity=1
- joint right_4C2_Joint1: limit lower=0 upper=0.82 effort=1 velocity=1 -> lower=0 upper=0.82 effort=50 velocity=1
- joint right_4C2_Joint2: limit lower=0 upper=0.82 effort=1 velocity=1 -> lower=0 upper=0.82 effort=50 velocity=1
- joint right_4C2_Joint3: limit lower=-0.82 upper=0 effort=1 velocity=1 -> lower=-0.82 upper=0 effort=50 velocity=1
- joint right_4C2_Joint4: limit lower=-0.82 upper=0 effort=1 velocity=1 -> lower=-0.82 upper=0 effort=50 velocity=1
- joint right_4C2_Joint5: limit lower=0 upper=0.82 effort=1 velocity=1 -> lower=0 upper=0.82 effort=50 velocity=1
- joint right_4C2_Joint6: limit lower=0 upper=0.82 effort=1 velocity=1 -> lower=0 upper=0.82 effort=50 velocity=1
